Commit message: Puzzlebot doing circular trajectory in RVIZ. Part1/2 completed. No control.

File: urdf/puzzlebot_jetson_ed_urdf.urdf (robot description, URDF)
Before this commit: robot Puzzlebot Jetson-Lidar Ed., 2 links, 1 joints
Links:
- added link wl_link, mass 0.01; collision mesh filename=package://localisation/models/MCR2_1000_1_1_Wheel_Coupler_2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; visual mesh filename=package://localisation/models/MCR2_1000_1_1_Wheel_Coupler_2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
- added link wr_link, mass 0.01; collision mesh filename=package://localisation/models/MCR2_1000_1_1_Wheel_Coupler_2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; visual mesh filename=package://localisation/models/MCR2_1000_1_1_Wheel_Coupler_2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
Joints:
- added joint leftWheel: type continuous, parent chassis, child wl_link, origin xyz=0.0 0.0 0.05
- added joint rightWheel: type continuous, parent chassis, child wr_link, origin xyz=0.0 0.0 0.05

Commit message: Puzzlebot finally moving correctly with the wheels attached.

File: urdf/puzzlebot_jetson_ed_urdf.urdf (robot description, URDF)
Before this commit: robot Puzzlebot Jetson-Lidar Ed., 4 links, 3 joints
Links:
- added link camera_link; visual mesh filename=package://localisation/models/camera.stl
- link wl_link: mass 0.01 -> None; geometry visual mesh filename=package://localisation/models/MCR2_1000_1_1_Wheel_Coupler_2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
- link wr_link: mass 0.01 -> None; geometry visual mesh filename=package://localisation/models/MCR2_1000_1_1_Wheel_Coupler_2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
Joints:
- added joint camera_joint: type fixed, parent chassis, child camera_link, origin xyz=0.045 0 0.02
- joint leftWheel: axis (none) -> 0 1 0; origin xyz=0.0 0.0 0.05 -> xyz=0.0525 0.103 0.05 rpy=0 0.0 0.0
- joint rightWheel: axis (none) -> 0 1 0; origin xyz=0.0 0.0 0.05 -> xyz=0.0525 -1.00 0.0
